File: earring.kicad_sch (KiCad schematic)
At the start: 106 parts, among them J2 USB_C_Receptacle_USB2.0, Q1 NMOS 20V 0.75A 500mΩ@4.5V, Q2 NMOS 20V 0.75A 500mΩ@4.5V, Q3 NMOS 20V 0.75A 500mΩ@4.5V, Q4 NMOS 20V 0.75A 500mΩ@4.5V, Q5 light_sensor, U1 Magnetic Switch, U10 USBLC6-2P6, U20 LGS4056H, U24 SK9822-EC20, U3 RP2040, U4 W25Q16JV, U6 Buffer, U7 LSM6DS3, U9 NCP730BMT330TBG, Y1 Crystal_GND24

Commit message: rework power control to simplify and remove VBAT from MCU pins
Parts:
- removed Q1, Q2, Q3, Q4: NMOS 20V 0.75A 500mΩ@4.5V, Package_DFN_QFN:Diodes_DFN1006-3, symbol Device:Q_NMOS_GSD
- added U43, U44: TPS22913BYZVR, footprints:YZV0004ADAD, symbol 2024-12-11_08-06-17:TPS22913BYZVR
- R10: value 20k -> 10k; LCSC C25765 -> C25804
- U4: value W25Q16JV -> W25Q16JVUXIQ
- U8: value ~ -> DS6091AED4
Connections:
- net LED_1_GND is gone; now on net GND: C27.2, C28.2, U16.2 (GND), U17.2 (GND), U18.2 (GND), U19.2 (GND), U21.2 (GND), U22.2 (GND), U48.2 (GND), U49.2 (GND), U52.2 (GND)
- net LED_2_GND is gone; now on net GND: C31.2, C32.2, C33.2, R8.2, U27.2 (GND), U28.2 (GND), U29.2 (GND), U30.2 (GND), U34.2 (GND), U35.2 (GND), U36.2 (GND), U37.2 (GND), U41.2 (GND), U42.2 (GND), U50.2 (GND)
- net LED_3_GND is gone; now on net GND: C29.2, C30.2, U24.2 (GND), U25.2 (GND), U26.2 (GND), U31.2 (GND), U32.2 (GND), U33.2 (GND), U38.2 (GND), U39.2 (GND), U40.2 (GND)
- net LED_4_GND is gone; now on net GND: C25.2, C26.2, R12.1, U11.2 (GND), U12.2 (GND), U13.2 (GND), U14.2 (GND), U15.2 (GND), U45.2 (GND), U46.2 (GND), U47.2 (GND), U5.2 (GND)
- net +3V3: no longer Q5.1
- net +BATT: now also U43.A2 (VIN), U44.A2 (VIN); no longer C25.1, C26.1, C27.1, C28.1, C29.1, C30.1, C31.1, C32.1, R11.2, U11.5 (VDD), U12.5 (VDD), U13.5 (VDD), U14.5 (VDD), U15.5 (VDD), U16.5 (VDD), U17.5 (VDD), U18.5 (VDD), U19.5 (VDD), U21.5 (VDD), U22.5 (VDD), U24.5 (VDD), U25.5 (VDD), U26.5 (VDD), U27.5 (VDD), U28.5 (VDD), U29.5 (VDD), U30.5 (VDD), U31.5 (VDD), U32.5 (VDD), U33.5 (VDD), U34.5 (VDD), U35.5 (VDD), U36.5 (VDD), U37.5 (VDD), U38.5 (VDD), U39.5 (VDD), U40.5 (VDD), U41.5 (VDD), U42.5 (VDD), U45.5 (VDD), U46.5 (VDD), U47.5 (VDD), U48.5 (VDD), U49.5 (VDD), U5.5 (VDD), U50.5 (VDD), U52.5 (VDD)
- net GND: now also U43.B1 (GND), U44.B1 (GND)
- net QSPI_SCLK: no longer R1.1
- net QSPI_SS: now also R1.1
- net SW_LED_1: now also U43.B2 (ON), U44.B2 (ON)
- net RUN renamed 3v3EN
- new net LED_1_V: C25.1, C26.1, C27.1, C28.1, C29.1, C30.1, C31.1, C32.1, Q5.1, R11.2, U11.5 (VDD), U12.5 (VDD), U13.5 (VDD), U14.5 (VDD), U15.5 (VDD), U16.5 (VDD), U17.5 (VDD), U18.5 (VDD), U19.5 (VDD), U21.5 (VDD), U22.5 (VDD), U24.5 (VDD), U25.5 (VDD), U26.5 (VDD), U27.5 (VDD), U28.5 (VDD), U29.5 (VDD), U30.5 (VDD), U31.5 (VDD), U32.5 (VDD), U33.5 (VDD), U34.5 (VDD), U35.5 (VDD), U36.5 (VDD), U37.5 (VDD), U38.5 (VDD), U39.5 (VDD), U40.5 (VDD), U41.5 (VDD), U42.5 (VDD), U43.A1 (VOUT), U44.A1 (VOUT), U45.5 (VDD), U46.5 (VDD), U47.5 (VDD), U48.5 (VDD), U49.5 (VDD), U5.5 (VDD), U50.5 (VDD), U52.5 (VDD)
- no-connect marks 0 -> 4
Other:
- note added: "3v3EN high when no magnet present high = enabled"
- note added: "Calculated 20pf is good assuming 2pf stray capacitance"
- note added: "PG can be left floating"
- note added: "R10 sets charging current 10k = 100 ma"
- note added: "Temp floating is okay."
- note added: "Undervoltage cutoff 2.80v Overvoltage cutoff 4.30v"
- note added: "buffer flips at less than 0.7v should take 238ms for it to rise http://ladyada.net/library/rccalc.html"
- note added: "buffer is open collector"
- note removed: "R10 sets charging current 20k = 50 ma"
- note removed: "Run high when no magnet present"
- note removed: "TODO: TALK TO OPAL ABOUT CHARGE CURRENTS HERE"
- note removed: "VBATT THROUGH RESISTOR TO CPU OKAY WHEN CPU IS UNPOWERED?"
- note removed: "need to double check RC rise time considering buffer flips at less than 0.7v"
- moved on the sheet: C25, C26, C29, C30, R1, R11, R12

Commit message: check in complex startup circuit before simplification
Parts:
- removed C24: 100n, Capacitor_SMD:C_0402_1005Metric, symbol Device:C
- removed D2: D, Diode_SMD:D_SOD-523, symbol Device:D
- removed U6: Buffer, digikey-footprints:UFDFN-6_1.45x1mm, symbol earring:SN74LVC1G07-DFN6
- added D1, D4, D5: D, Diode_SMD:D_SOD-882, symbol Device:D
- added D2, D3, D6: 3.3v Zener, Diode_SMD:D_SOD-882, symbol Device:D_Zener
- added Q1, Q2: BSS214NW, Package_DFN_QFN:Diodes_DFN1006-3, symbol Transistor_FET:BSS214NW
- added R13, R15, R16: 100k, Resistor_SMD:R_0402_1005Metric, symbol Device:R
- added R17: 1M, Resistor_SMD:R_0402_1005Metric, symbol Device:R
- added R18, R20: 10k, Resistor_SMD:R_0402_1005Metric, symbol Device:R
- R2: value 100k -> 10k
Connections:
- net +3V3: now also R15.1; no longer R2.1, U3.26 (RUN)
- net +BATT: now also R13.1
- net 3v3EN: now also D3.2 (A), D5.1 (K), R13.2, R18.1; no longer U1.2 (VOUT)
- net GND: now also D2.2 (A), Q1.2 (S), Q2.2 (S); no longer C3.2
- net VBUS: now also R2.2, D4.2 (A)
- net ~{USB_BOOT}: now also D1.2 (A)
- net mag: now reaches C3.1
- net mag: now also U1.2 (VOUT), Q1.1 (G), R20.1; no longer R2.2
- net SW_LED_3 renamed ENA_GPIO
- net ENA_GPIO: now also D5.2 (A)
- net SW_LED_4 renamed RUN_GPIO
- new net: Q1.3 (D), R18.2
- new net: C3.2, R16.1, R2.1
- new net: Q2.3 (D), R15.2
- new net: D2.1 (K), R20.2
- new net: D3.1 (K), D4.1 (K)
- new net RUN: U3.26 (RUN)
Other:
- note added: "///"
- note added: "0.9 volt activation threshold"
- note added: "0.9v high threshold"
- note added: "1.7 volts"
- note added: "3.3v"
- note added: "3V3EN"
- note added: "BATTERY"
- note added: "DELAYED HIGH"
- note added: "Don't backfeed to vbus or usb_boot circuit fails"
- note added: "HIGH"
- note added: "HIGH BY MCU"
- note added: "LOW"
- note added: "MAG"
- note added: "MAG RELEASE"
- note added: "MAG TAP"
- note added: "NO MAG"
- note added: "Prevent vbus from overvoltage on BATT or 3v3EN"
- note added: "RUN"
- note added: "USB POWER"
- note added: "USBBOOT"
- note added: "VBAT"
- note removed: "buffer is open collector"
- note removed: "must stay low for longer than 100us"
- moved on the sheet: C19, U1

Commit message: simplify power and boot circuit
Parts:
- removed C3: 10u, Capacitor_SMD:C_0402_1005Metric, symbol Device:C
- removed D2, D3, D6: 3.3v Zener, Diode_SMD:D_SOD-882, symbol Device:D_Zener
- removed D5: D, Diode_SMD:D_SOD-882, symbol Device:D
- removed Q1, Q2: BSS214NW, Package_DFN_QFN:Diodes_DFN1006-3, symbol Transistor_FET:BSS214NW
- removed R15, R16: 100k, Resistor_SMD:R_0402_1005Metric, symbol Device:R
- removed R17: 1M, Resistor_SMD:R_0402_1005Metric, symbol Device:R
- removed R18, R2, R20: 10k, Resistor_SMD:R_0402_1005Metric, symbol Device:R
- added TP7, TP8: TestPoint, TestPoint:TestPoint_Pad_D1.0mm, symbol Connector:TestPoint
Connections:
- net RUN is gone; now on net +3V3: U3.26 (RUN)
- net +BATT: no longer R13.1
- net 3v3EN: now also D1.1 (K), D4.1 (K); no longer R13.2
- net GND: now also TP8.1
- net VBUS: now also D1.2 (A); no longer D4.2 (A)
- net ~{USB_BOOT}: now also TP7.1; no longer D1.2 (A)
- net mag: no longer names the net of U1.2 (VOUT)
- net mag: now also R13.1
- new net: D4.2 (A), R13.2
Other:
- note removed: "Magnet sends signal low"
- moved on the sheet: C19, D4, R13, U1

Commit message: pcb files seem possibly ready to order
Parts:
- R10: LCSC C25804 -> C60490
- U24: value SK9822-EC20 -> ~
Connections:
- net ENA_GPIO: no longer names the net of U3.2 (GPIO0)
- net RUN_GPIO: no longer names the net of U3.3 (GPIO1)
- net SW_LED_2: no longer names the net of U3.35 (GPIO23)
- no-connect marks 4 -> 29
Other:
- note removed: "///"
- note removed: "0.9v high threshold"
- note removed: "1.7 volts"
- note removed: "3.3v"
- note removed: "3V3EN"
- note removed: "BATTERY"
- note removed: "DELAYED HIGH"
- note removed: "HIGH"
- note removed: "HIGH BY MCU"
- note removed: "LOW"
- note removed: "MAG"
- note removed: "MAG RELEASE"
- note removed: "MAG TAP"
- note removed: "NO MAG"
- note removed: "RUN"
- note removed: "USB POWER"
- note removed: "USBBOOT"
- note removed: "VBAT"
- moved on the sheet: C1, C10, C11, C12, C13, C14, C15, C16, C17, C18, C19, C23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

Commit message: about to rewire
Other:
- note removed: "Calculated 20pf is good assuming 2pf stray capacitance"
- moved on the sheet: C14, C17, C18, C27, C28, U24, U25, U26, U31, U32, U33, U38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

Commit message: Fixed power circuit and ordered June 2025
Parts:
- removed D1, D4: D, Diode_SMD:D_SOD-882, symbol Device:D
- added Q1: Q_NMOS_SGD, parts2:DFN1006-3L_L1.0-W0.6-BL, symbol Device:Q_NMOS_SDG
- added R15, R2: 10k, Resistor_SMD:R_0402_1005Metric, symbol Device:R
- C4: value 100n -> 10u; LCSC C60474 -> C315248
- C5, C6: value 20p -> 12p; LCSC C107000 -> C1547
Connections:
- net +BATT: now also R13.2
- net 3v3EN: now also R15.2, R2.2
- net CHRG: now also U20.7 (CHRG), U3.28 (GPIO17); no longer U20.6 (Done), U3.27 (GPIO16)
- net DONE: now also U20.6 (Done), U3.27 (GPIO16); no longer U20.7 (CHRG), U3.28 (GPIO17)
- net GND: now also Q1.1 (S)
- net LED_SCK_2: now also U45.4 (CKL); no longer U41.4 (CKL)
- net LED_TX_2: now also U45.3 (SDI); no longer U41.3 (SDI)
- net VBUS: now also R2.1
- net at R13.1: now also Q1.2 (D), R15.1; no longer U1.2 (VOUT)
- net at U12.1 (SDO): now also U38.3 (SDI)
- net at U12.6 (CKO): now also U38.4 (CKL)
- net at U18.1 (SDO): now also U41.3 (SDI)
- net at U18.6 (CKO): now also U41.4 (CKL)
- net LED_SCK_3: no longer names the net of U3.37 (GPIO25)
- net LED_SCK_3: no longer U38.4 (CKL)
- net LED_SCK_4: no longer names the net of U3.40 (GPIO28_ADC2)
- net LED_SCK_4: no longer U45.4 (CKL)
- net LED_TX_3: no longer names the net of U3.36 (GPIO24)
- net LED_TX_3: no longer U38.3 (SDI)
- net LED_TX_4: no longer names the net of U3.39 (GPIO27_ADC1)
- net LED_TX_4: no longer U45.3 (SDI)
- new net: Q1.3 (G), U1.2 (VOUT)
Other:
- note added: "high = enabled"
- note added: "high when no magnet present low when magnet present"
- note removed: "3v3EN high when no magnet present high = enabled"
- moved on the sheet: R13, U24, U25, U26, U31, U32, U33, U38, U39, U40, U44

Commit message: more clean up. looking pretty good
Parts:
- removed C13: 100n, Capacitor_SMD:C_0402_1005Metric, symbol Device:C
- C1: value 100n -> 1u; LCSC C60474 -> C29266
Changed lines of the file:
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@@
 	)
 	(junction
-		(at 208.28 78.74)
-		(diameter 0)
-		(color 0 0 0 0)
-	)
-	(junction
 		(at 68.58 153.67)
 		(diameter 0)
@@
 	)
 	(junction
-		(at 208.28 90.17)
-		(diameter 0)
-		(color 0 0 0 0)
-	)
-	(junction
 		(at 86.36 142.24)
 		(diameter 0)
@@
 	(wire
 		(pts
-			(xy 199.39 78.74) (xy 208.28 78.74)
-		)
-		(stroke
-			(width 0)
-			(type default)
-		)
-	)
-	(wire
-		(pts
 			(xy 414.02 66.04) (xy 411.48 66.04)
 		)
@@
 	(wire
 		(pts
-			(xy 208.28 87.63) (xy 208.28 90.17)
-		)
-		(stroke
-			(width 0)
-			(type default)
-		)
-	)
-	(wire
-		(pts
 			(xy 212.09 63.5) (xy 222.25 63.5)
 		)
@@
 	(wire
 		(pts
-			(xy 208.28 90.17) (xy 214.63 90.17)
-		)
-		(stroke
-			(width 0)
-			(type default)
-		)
-	)
-	(wire
-		(pts
 			(xy 361.95 201.93) (xy 425.45 201.93)
 		)
@@
 	(wire
 		(pts
-			(xy 208.28 80.01) (xy 208.28 78.74)
-		)
-		(stroke
-			(width 0)
-			(type default)
-		)
-	)
-	(wire
-		(pts
-			(xy 199.39 90.17) (xy 208.28 90.17)
+			(xy 199.39 90.17) (xy 214.63 90.17)
 		)
 		(stroke
@@
 	(wire
 		(pts
-			(xy 208.28 78.74) (xy 214.63 78.74)
+			(xy 199.39 78.74) (xy 214.63 78.74)
 		)
 		(stroke
@@
 			)
 		)
-		(property "Value" "100n"
+		(property "Value" "1u"
 			(at 49.911 223.393 0)
 			(effects
@@
 			)
 		)
-		(property "LCSC" "C60474"
+		(property "LCSC" "C29266"
 			(at 46.99 222.25 0)
 			(effects
@@
 					(unit 1)
 				)
-			)
-		)
-	)
-	(symbol
-		(lib_id "Device:C")
-		(at 208.28 83.82 0)
-		(unit 1)
-		(exclude_from_sim no)
-		(in_bom yes)
-		(on_board yes)
-		(dnp no)
-		(property "Reference" "C13"
-			(at 204.089 81.7626 0)
-			(effects
-				(font
-					(size 1.27 1.27)
-				)
-				(justify left)
-			)
-		)
-		(property "Value" "100n"
-			(at 208.534 85.852 0)
-			(effects
-				(font
-					(size 1.27 1.27)
-				)
-				(justify left)
-			)
-		)
-		(property "Footprint" "Capacitor_SMD:C_0402_1005Metric"
-			(at 209.2452 87.63 0)
-			(effects
-				(font
-					(size 1.27 1.27)
-				)
-				(hide yes)
-			)
-		)
-		(property "Datasheet" "~"
-			(at 208.28 83.82 0)
-			(effects
-				(font
-					(size 1.27 1.27)
-				)
-				(hide yes)
-			)
-		)
-		(property "Description" ""
-			(at 208.28 83.82 0)
-			(effects
-				(font
-					(size 1.27 1.27)
-				)
-				(hide yes)
-			)
-		)
-		(property "LCSC" "C60474"
-			(at 208.28 83.82 0)
-			(effects
-				(font
-					(size 1.27 1.27)
-				)
-				(hide yes)
-			)
-		)
-		(pin "1"
-		)
-		(pin "2"
-		)
-		(instances
-			(project "earring"
-				(path "/10ff4ace-8dac-45ce-94a5-ae8ae7d42914"
-					(reference "C13")
-					(unit 1)
-				)
